File: choc/single-choc.kicad_pcb (KiCad board)
At the start: 2 copper layers, 97 x 117 mm, 241 parts, among them J1 Conn_01x01, J10 Conn_01x01, J100 Conn_01x01, J101 Conn_01x01, J102 Conn_01x01, J103 Conn_01x01, J104 Conn_01x01, J105 Conn_01x01, J106 Conn_01x01, J107 Conn_01x01, J108 Conn_01x01, J109 Conn_01x01, J11 Conn_01x01, J110 Conn_01x01, J111 Conn_01x01, J112 Conn_01x01, J113 Conn_01x01, J114 Conn_01x01, J115 Conn_01x01, J116 Conn_01x01, J117 Conn_01x01, J118 Conn_01x01, J119 Conn_01x01, J12 Conn_01x01, J120 Conn_01x01, J121 Conn_01x01, J122 Conn_01x01, J123 Conn_01x01, J124 Conn_01x01, J125 Conn_01x01, J126 Conn_01x01, J127 Conn_01x01, J128 Conn_01x01, J129 Conn_01x01, J13 Conn_01x01, J130 Conn_01x01, J131 Conn_01x01, J132 Conn_01x01, J133 Conn_01x01, J134 Conn_01x01, J135 Conn_01x01, J136 Conn_01x01, J137 Conn_01x01, J138 Conn_01x01, J139 Conn_01x01, J14 Conn_01x01, J140 Conn_01x01, J141 Conn_01x01, J142 Conn_01x01, J143 Conn_01x01, J144 Conn_01x01, J145 Conn_01x01, J146 Conn_01x01, J147 Conn_01x01, J148 Conn_01x01, J149 Conn_01x01, J15 Conn_01x01, J150 Conn_01x01, J151 Conn_01x01, J152 Conn_01x01, J153 Conn_01x01, J154 Conn_01x01, J155 Conn_01x01, J156 Conn_01x01, J157 Conn_01x01, J158 Conn_01x01, J159 Conn_01x01, J16 Conn_01x01, J160 Conn_01x01, J161 Conn_01x01, J162 Conn_01x01, J163 Conn_01x01, J164 Conn_01x01, J165 Conn_01x01, J166 Conn_01x01, J167 Conn_01x01, J168 Conn_01x01, J169 Conn_01x01, J17 Conn_01x01, J170 Conn_01x01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

Commit message: finished
Parts:
- added Ref**: Val**, footprints:hole-four, F.Cu at (38.5, 32.0)
- added Ref**: Val**, footprints:hole-three, F.Cu at (23.2, 81.2)
- added Ref**: Val**, footprints:hole-four, F.Cu at (38.5, 112.0)
- added Ref**: Val**, footprints:hole-three, F.Cu at (23.2, 101.2)
- added Ref**: Val**, footprints:hole-three, F.Cu at (23.2, 118.5)
- added Ref**: Val**, footprints:hole-four, F.Cu at (38.5, 132.0)
- added Ref**: Val**, footprints:hole-three, F.Cu at (23.2, 121.2)
- added Ref**: Val**, footprints:hole-three, F.Cu at (103.2, 121.2)
- added Ref**: Val**, footprints:hole-four, F.Cu at (101.5, 132.0)
- added Ref**: Val**, footprints:hole-three, F.Cu at (103.2, 101.2)
- added Ref**: Val**, footprints:hole-three, F.Cu at (103.2, 118.5)
- added Ref**: Val**, footprints:hole-four, F.Cu at (38.5, 52.0)
- added Ref**: Val**, footprints:hole-four, F.Cu at (101.5, 112.0)
- added Ref**: Val**, footprints:hole-three, F.Cu at (103.2, 98.5)
- added Ref**: Val**, footprints:hole-four, F.Cu at (101.5, 92.0)
- added Ref**: Val**, footprints:hole-three, F.Cu at (103.2, 81.2)
- added Ref**: Val**, footprints:hole-three, F.Cu at (103.2, 61.2)
- added Ref**: Val**, footprints:hole-three, F.Cu at (103.2, 78.5)
- added Ref**: Val**, footprints:hole-four, F.Cu at (101.5, 72.0)
- added Ref**: Val**, footprints:hole-four, F.Cu at (101.5, 52.0)
- added Ref**: Val**, footprints:hole-three, F.Cu at (103.2, 58.5)
- added Ref**: Val**, footprints:hole-three, F.Cu at (103.2, 41.2)
- added Ref**: Val**, footprints:hole-three, F.Cu at (23.2, 58.5)
- added Ref**: Val**, footprints:hole-four, F.Cu at (101.5, 32.0)
- added Ref**: Val**, footprints:hole-three, F.Cu at (103.2, 38.5)
- added Ref**: Val**, footprints:hole-four, F.Cu at (81.5, 32.0)
- added Ref**: Val**, footprints:hole-three, F.Cu at (83.2, 38.5)
- added Ref**: Val**, footprints:hole-four, F.Cu at (98.5, 32.0)
- added Ref**: Val**, footprints:hole-four, F.Cu at (78.5, 32.0)
- added Ref**: Val**, footprints:hole-four, F.Cu at (61.5, 32.0)
- added Ref**: Val**, footprints:hole-three, F.Cu at (63.2, 38.5)
- added Ref**: Val**, footprints:hole-three, F.Cu at (43.2, 38.5)
- added Ref**: Val**, footprints:hole-four, F.Cu at (41.5, 32.0)
- added Ref** (x2): Val**, footprints:hole-three, F.Cu at (23.2, 41.2)
- added Ref**: Val**, footprints:hole-four, F.Cu at (58.5, 32.0)
- added Ref**: Val**, footprints:hole-three, F.Cu at (63.2, 101.2)
- added Ref**: Val**, footprints:hole-four, F.Cu at (61.5, 112.0)
- added Ref**: Val**, footprints:hole-three, F.Cu at (63.2, 118.5)
- added Ref**: Val**, footprints:hole-four, F.Cu at (78.5, 112.0)
- added Ref**: Val**, footprints:hole-four, F.Cu at (78.5, 92.0)
- added Ref**: Val**, footprints:hole-three, F.Cu at (63.2, 98.5)
- added Ref**: Val**, footprints:hole-four, F.Cu at (61.5, 92.0)
- added Ref**: Val**, footprints:hole-three, F.Cu at (63.2, 81.2)
- added Ref**: Val**, footprints:hole-four, F.Cu at (78.5, 72.0)
- added Ref**: Val**, footprints:hole-four, F.Cu at (38.5, 72.0)
- added Ref**: Val**, footprints:hole-three, F.Cu at (63.2, 78.5)
- added Ref**: Val**, footprints:hole-four, F.Cu at (61.5, 72.0)
- added Ref**: Val**, footprints:hole-three, F.Cu at (63.2, 61.2)
- added Ref**: Val**, footprints:hole-four, F.Cu at (78.5, 52.0)
- added Ref**: Val**, footprints:hole-three, F.Cu at (63.2, 58.5)
- added Ref**: Val**, footprints:hole-four, F.Cu at (61.5, 52.0)
- added Ref**: Val**, footprints:hole-three, F.Cu at (63.2, 41.2)
- added Ref**: Val**, footprints:hole-four, F.Cu at (98.5, 52.0)
- added Ref**: Val**, footprints:hole-three, F.Cu at (83.2, 58.5)
- added Ref**: Val**, footprints:hole-four, F.Cu at (81.5, 52.0)
- added Ref**: Val**, footprints:hole-three, F.Cu at (23.2, 61.2)
- added Ref**: Val**, footprints:hole-three, F.Cu at (83.2, 41.2)
- added Ref**: Val**, footprints:hole-four, F.Cu at (81.5, 72.0)
- added Ref**: Val**, footprints:hole-three, F.Cu at (83.2, 78.5)
- added Ref**: Val**, footprints:hole-three, F.Cu at (83.2, 61.2)
- added Ref**: Val**, footprints:hole-four, F.Cu at (98.5, 72.0)
- added Ref**: Val**, footprints:hole-four, F.Cu at (81.5, 92.0)
- added Ref**: Val**, footprints:hole-three, F.Cu at (83.2, 81.2)
- added Ref**: Val**, footprints:hole-three, F.Cu at (83.2, 98.5)
- added Ref**: Val**, footprints:hole-four, F.Cu at (98.5, 92.0)
- added Ref**: Val**, footprints:hole-four, F.Cu at (98.5, 112.0)
- added Ref**: Val**, footprints:hole-three, F.Cu at (23.2, 78.5)
- added Ref**: Val**, footprints:hole-four, F.Cu at (81.5, 112.0)
- added Ref**: Val**, footprints:hole-three, F.Cu at (83.2, 101.2)
- added Ref**: Val**, footprints:hole-three, F.Cu at (83.2, 118.5)
- added Ref**: Val**, footprints:hole-four, F.Cu at (98.5, 132.0)
- added Ref**: Val**, footprints:hole-three, F.Cu at (83.2, 121.2)
- added Ref**: Val**, footprints:hole-four, F.Cu at (81.5, 132.0)
- added Ref**: Val**, footprints:hole-four, F.Cu at (78.5, 132.0)
- added Ref**: Val**, footprints:hole-three, F.Cu at (63.2, 121.2)
- added Ref**: Val**, footprints:hole-four, F.Cu at (61.5, 132.0)
- added Ref**: Val**, footprints:hole-three, F.Cu at (43.2, 121.2)
- added Ref**: Val**, footprints:hole-three, F.Cu at (23.2, 98.5)
- added Ref**: Val**, footprints:hole-four, F.Cu at (58.5, 132.0)
- added Ref**: Val**, footprints:hole-four, F.Cu at (41.5, 132.0)
- added Ref**: Val**, footprints:hole-three, F.Cu at (43.2, 101.2)
- added Ref**: Val**, footprints:hole-four, F.Cu at (58.5, 112.0)
- added Ref**: Val**, footprints:hole-three, F.Cu at (43.2, 118.5)
- added Ref**: Val**, footprints:hole-four, F.Cu at (41.5, 112.0)
- added Ref**: Val**, footprints:hole-three, F.Cu at (43.2, 81.2)
- added Ref**: Val**, footprints:hole-four, F.Cu at (41.5, 92.0)
- added Ref**: Val**, footprints:hole-four, F.Cu at (58.5, 92.0)
- added Ref**: Val**, footprints:hole-three, F.Cu at (43.2, 98.5)
- added Ref**: Val**, footprints:hole-four, F.Cu at (38.5, 92.0)
- added Ref**: Val**, footprints:hole-four, F.Cu at (41.5, 72.0)
- added Ref**: Val**, footprints:hole-four, F.Cu at (58.5, 72.0)
- added Ref**: Val**, footprints:hole-three, F.Cu at (43.2, 78.5)
- added Ref**: Val**, footprints:hole-three, F.Cu at (43.2, 61.2)
- added Ref**: Val**, footprints:hole-four, F.Cu at (58.5, 52.0)
- added Ref**: Val**, footprints:hole-four, F.Cu at (41.5, 52.0)
- added Ref**: Val**, footprints:hole-three, F.Cu at (43.2, 58.5)
- added Ref**: Val**, footprints:hole-three, F.Cu at (43.2, 41.2)
