File: standard/single-standard.kicad_pcb (KiCad board)
At the start: 2 copper layers, 89 x 89 mm, 240 parts, among them J1 Conn_01x01, J10 Conn_01x01, J100 Conn_01x01, J101 Conn_01x01, J102 Conn_01x01, J103 Conn_01x01, J104 Conn_01x01, J105 Conn_01x01, J106 Conn_01x01, J107 Conn_01x01, J108 Conn_01x01, J109 Conn_01x01, J11 Conn_01x01, J110 Conn_01x01, J111 Conn_01x01, J112 Conn_01x01, J113 Conn_01x01, J114 Conn_01x01, J115 Conn_01x01, J116 Conn_01x01, J117 Conn_01x01, J118 Conn_01x01, J119 Conn_01x01, J12 Conn_01x01, J120 Conn_01x01, J121 Conn_01x01, J122 Conn_01x01, J123 Conn_01x01, J124 Conn_01x01, J125 Conn_01x01, J126 Conn_01x01, J127 Conn_01x01, J128 Conn_01x01, J129 Conn_01x01, J13 Conn_01x01, J130 Conn_01x01, J131 Conn_01x01, J132 Conn_01x01, J133 Conn_01x01, J134 Conn_01x01, J135 Conn_01x01, J136 Conn_01x01, J137 Conn_01x01, J138 Conn_01x01, J139 Conn_01x01, J14 Conn_01x01, J140 Conn_01x01, J141 Conn_01x01, J142 Conn_01x01, J143 Conn_01x01, J144 Conn_01x01, J145 Conn_01x01, J146 Conn_01x01, J147 Conn_01x01, J148 Conn_01x01, J149 Conn_01x01, J15 Conn_01x01, J150 Conn_01x01, J151 Conn_01x01, J152 Conn_01x01, J153 Conn_01x01, J154 Conn_01x01, J155 Conn_01x01, J156 Conn_01x01, J157 Conn_01x01, J158 Conn_01x01, J159 Conn_01x01, J16 Conn_01x01, J160 Conn_01x01, J161 Conn_01x01, J162 Conn_01x01, J163 Conn_01x01, J164 Conn_01x01, J165 Conn_01x01, J166 Conn_01x01, J167 Conn_01x01, J168 Conn_01x01, J169 Conn_01x01, J17 Conn_01x01, J170 Conn_01x01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

Commit message: will jlc accept this shit? to be concluded.
Parts:
- moved J107 11.0 mm to (113.5, 116.0)
- moved J108 11.0 mm to (113.5, 126.0)
- moved J119 11.0 mm to (126.5, 116.0)
- moved J120 11.0 mm to (126.5, 126.0)
- moved J179 11.0 mm to (113.5, 120.0)
- moved J180 11.0 mm to (126.5, 120.0)
- moved diode30 11.0 mm to (120.0, 126.0)
- moved switch30 11.0 mm to (120.0, 122.5)
- moved J105 10.0 mm to (113.5, 99.5)
- moved J106 10.0 mm to (113.5, 109.5)
- moved J117 10.0 mm to (126.5, 99.5)
- moved J118 10.0 mm to (126.5, 109.5)
- moved J160 10.0 mm to (113.5, 103.5)
- moved J170 10.0 mm to (126.5, 103.5)
- moved diode29 10.0 mm to (120.0, 109.5)
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Routing:
- net Net-(J121-Pad1): track 122.9 -> 148.7 mm
- net Net-(J125-Pad1): track 122.9 -> 148.5 mm
- net Net-(J123-Pad1): track 122.9 -> 148.5 mm
- net Net-(J171-Pad1): track 122.9 -> 148.5 mm
- net Net-(J129-Pad1): track 122.9 -> 148.5 mm
- net Net-(J127-Pad1): track 122.9 -> 148.5 mm
- net Net-(J73-Pad1): track 255.5 -> 251.7 mm
- net Net-(J49-Pad1): track 255.5 -> 251.7 mm
- net Net-(J1-Pad1): track 255.7 -> 252.0 mm
- net Net-(J100-Pad1): track 255.5 -> 252.0 mm
- net Net-(J25-Pad1): track 255.5 -> 252.0 mm
Other:
- board size 89 x 89 mm -> 97 x 96 mm

Commit message: please let this one through, jlc.
Parts:
- added Ref**: Val**, footprints:hole-two, F.Cu at (111.5, 87.0)
- added Ref**: Val**, footprints:hole-two, F.Cu at (108.5, 37.5)
- added Ref**: Val**, footprints:hole-two, F.Cu at (111.5, 37.5)
- added Ref**: Val**, footprints:hole-two, F.Cu at (108.5, 120.0)
- added Ref**: Val**, footprints:hole-two, F.Cu at (88.5, 37.5)
- added Ref**: Val**, footprints:hole-two, F.Cu at (91.5, 87.0)
- added Ref**: Val**, footprints:hole-two, F.Cu at (91.5, 54.0)
- added Ref**: Val**, footprints:hole-two, F.Cu at (88.5, 54.0)
- added Ref**: Val**, footprints:hole-two, F.Cu at (91.5, 70.5)
- added Ref**: Val**, footprints:hole-two, F.Cu at (88.5, 103.5)
- added Ref**: Val**, footprints:hole-two, F.Cu at (91.5, 37.5)
- added Ref**: Val**, footprints:hole-two, F.Cu at (111.5, 70.5)
- added Ref**: Val**, footprints:hole-two, F.Cu at (88.5, 87.0)
- added Ref**: Val**, footprints:hole-two, F.Cu at (91.5, 103.5)
- added Ref**: Val**, footprints:hole-two, F.Cu at (88.5, 120.0)
- added Ref**: Val**, footprints:hole-two, F.Cu at (88.5, 70.5)
- added Ref**: Val**, footprints:hole-two, F.Cu at (91.5, 120.0)
- added Ref**: Val**, footprints:hole-two, F.Cu at (68.5, 37.5)
- added Ref**: Val**, footprints:hole-two, F.Cu at (71.5, 103.5)
- added Ref**: Val**, footprints:hole-two, F.Cu at (68.5, 120.0)
- added Ref**: Val**, footprints:hole-two, F.Cu at (71.5, 120.0)
- added Ref**: Val**, footprints:hole-two, F.Cu at (68.5, 70.5)
- added Ref**: Val**, footprints:hole-two, F.Cu at (108.5, 54.0)
- added Ref**: Val**, footprints:hole-two, F.Cu at (71.5, 87.0)
- added Ref**: Val**, footprints:hole-two, F.Cu at (68.5, 87.0)
- added Ref**: Val**, footprints:hole-two, F.Cu at (68.5, 103.5)
- added Ref**: Val**, footprints:hole-two, F.Cu at (68.5, 54.0)
- added Ref**: Val**, footprints:hole-two, F.Cu at (71.5, 70.5)
- added Ref**: Val**, footprints:hole-two, F.Cu at (71.5, 54.0)
- added Ref**: Val**, footprints:hole-two, F.Cu at (71.5, 37.5)
- added Ref**: Val**, footprints:hole-two, F.Cu at (51.5, 120.0)
- added Ref**: Val**, footprints:hole-two, F.Cu at (48.5, 120.0)
- added Ref**: Val**, footprints:hole-two, F.Cu at (51.5, 103.5)
- added Ref**: Val**, footprints:hole-two, F.Cu at (111.5, 120.0)
- added Ref**: Val**, footprints:hole-two, F.Cu at (48.5, 103.5)
- added Ref**: Val**, footprints:hole-two, F.Cu at (48.5, 87.0)
- added Ref**: Val**, footprints:hole-two, F.Cu at (51.5, 87.0)
- added Ref**: Val**, footprints:hole-two, F.Cu at (48.5, 70.5)
- added Ref**: Val**, footprints:hole-two, F.Cu at (51.5, 70.5)
- added Ref**: Val**, footprints:hole-two, F.Cu at (48.5, 54.0)
- added Ref**: Val**, footprints:hole-two, F.Cu at (51.5, 54.0)
- added Ref**: Val**, footprints:hole-two, F.Cu at (51.5, 37.5)
- added Ref**: Val**, footprints:hole-two, F.Cu at (48.5, 37.5)
- added Ref**: Val**, footprints:hole-three, F.Cu at (73.5, 114.0)
- added Ref**: Val**, footprints:hole-two, F.Cu at (108.5, 103.5)
- added Ref**: Val**, footprints:hole-three, F.Cu at (93.5, 111.0)
- added Ref**: Val**, footprints:hole-three, F.Cu at (53.5, 111.0)
- added Ref**: Val**, footprints:hole-three, F.Cu at (113.5, 114.0)
- added Ref**: Val**, footprints:hole-three, F.Cu at (113.5, 111.0)
- added Ref**: Val**, footprints:hole-three, F.Cu at (33.5, 111.0)
- added Ref**: Val**, footprints:hole-three, F.Cu at (33.5, 114.0)
- added Ref**: Val**, footprints:hole-three, F.Cu at (93.5, 114.0)
- added Ref**: Val**, footprints:hole-three, F.Cu at (73.5, 111.0)
- added Ref**: Val**, footprints:hole-three, F.Cu at (53.5, 114.0)
- added Ref**: Val**, footprints:hole-three, F.Cu at (73.5, 97.5)
- added Ref**: Val**, footprints:hole-two, F.Cu at (108.5, 87.0)
- added Ref**: Val**, footprints:hole-three, F.Cu at (33.5, 94.5)
- added Ref**: Val**, footprints:hole-three, F.Cu at (73.5, 94.5)
- added Ref**: Val**, footprints:hole-three, F.Cu at (113.5, 97.5)
- added Ref**: Val**, footprints:hole-three, F.Cu at (93.5, 97.5)
- added Ref**: Val**, footprints:hole-three, F.Cu at (113.5, 94.5)
- added Ref**: Val**, footprints:hole-three, F.Cu at (53.5, 97.5)
- added Ref**: Val**, footprints:hole-three, F.Cu at (33.5, 97.5)
- added Ref**: Val**, footprints:hole-three, F.Cu at (53.5, 94.5)
- added Ref**: Val**, footprints:hole-three, F.Cu at (93.5, 94.5)
- added Ref**: Val**, footprints:hole-three, F.Cu at (73.5, 81.0)
- added Ref**: Val**, footprints:hole-two, F.Cu at (108.5, 70.5)
- added Ref**: Val**, footprints:hole-three, F.Cu at (113.5, 78.0)
- added Ref**: Val**, footprints:hole-three, F.Cu at (33.5, 78.0)
- added Ref**: Val**, footprints:hole-three, F.Cu at (33.5, 81.0)
- added Ref**: Val**, footprints:hole-three, F.Cu at (53.5, 78.0)
- added Ref**: Val**, footprints:hole-three, F.Cu at (93.5, 81.0)
- added Ref**: Val**, footprints:hole-three, F.Cu at (113.5, 81.0)
- added Ref**: Val**, footprints:hole-three, F.Cu at (53.5, 81.0)
- added Ref**: Val**, footprints:hole-three, F.Cu at (93.5, 78.0)
- added Ref**: Val**, footprints:hole-three, F.Cu at (73.5, 78.0)
- added Ref**: Val**, footprints:hole-three, F.Cu at (33.5, 64.5)
- added Ref**: Val**, footprints:hole-two, F.Cu at (111.5, 54.0)
- added Ref**: Val**, footprints:hole-three, F.Cu at (53.5, 61.5)
- added Ref**: Val**, footprints:hole-three, F.Cu at (113.5, 64.5)
- added Ref**: Val**, footprints:hole-three, F.Cu at (113.5, 61.5)
- added Ref**: Val**, footprints:hole-three, F.Cu at (33.5, 61.5)
- added Ref**: Val**, footprints:hole-three, F.Cu at (73.5, 61.5)
- added Ref**: Val**, footprints:hole-three, F.Cu at (53.5, 64.5)
- added Ref**: Val**, footprints:hole-three, F.Cu at (93.5, 64.5)
- added Ref**: Val**, footprints:hole-three, F.Cu at (93.5, 61.5)
- added Ref**: Val**, footprints:hole-three, F.Cu at (73.5, 64.5)
- added Ref**: Val**, footprints:hole-three, F.Cu at (113.5, 48.0)
- added Ref**: Val**, footprints:hole-two, F.Cu at (111.5, 103.5)
- added Ref**: Val**, footprints:hole-three, F.Cu at (113.5, 45.0)
- added Ref**: Val**, footprints:hole-three, F.Cu at (93.5, 45.0)
- added Ref**: Val**, footprints:hole-three, F.Cu at (93.5, 48.0)
- added Ref**: Val**, footprints:hole-three, F.Cu at (73.5, 45.0)
- added Ref**: Val**, footprints:hole-three, F.Cu at (73.5, 48.0)
- added Ref**: Val**, footprints:hole-three, F.Cu at (53.5, 48.0)
- added Ref**: Val**, footprints:hole-three, F.Cu at (53.5, 45.0)
- added Ref**: Val**, footprints:hole-three, F.Cu at (33.5, 48.0)
- added Ref**: Val**, footprints:hole-three, F.Cu at (33.5, 45.0)
Routing:
- net Net-(J73-Pad1): track 251.7 -> 259.1 mm
- net Net-(J49-Pad1): track 251.7 -> 259.2 mm
- net Net-(J100-Pad1): track 252.0 -> 259.4 mm
- net Net-(J25-Pad1): track 252.0 -> 259.0 mm
- net Net-(J1-Pad1): track 252.0 -> 258.0 mm
Other:
- outline, holes or cut-outs redrawn

Commit message: larger snappy hole thingy.
Parts:
- moved Ref** 0.25 mm to (73.8, 114.0)
- moved Ref** 0.25 mm to (93.8, 111.0)
- moved Ref** 0.25 mm to (53.8, 111.0)
- moved Ref** 0.25 mm to (113.8, 114.0)
- moved Ref** 0.25 mm to (113.8, 111.0)
- moved Ref** 0.25 mm to (33.8, 111.0)
- moved Ref** 0.25 mm to (33.8, 114.0)
- moved Ref** 0.25 mm to (93.8, 114.0)
- moved Ref** 0.25 mm to (73.8, 111.0)
- moved Ref** 0.25 mm to (53.8, 114.0)
- moved Ref** 0.25 mm to (73.8, 97.5)
- moved Ref** 0.25 mm to (33.8, 94.5)
- moved Ref** 0.25 mm to (73.8, 94.5)
- moved Ref** 0.25 mm to (113.8, 97.5)
- moved Ref** 0.25 mm to (93.8, 97.5)
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
Commit message: wat?
Routing:
- added copper zone on B.Cu, net (none)
- added copper zone on F.Cu, net (none)
