File: socketsmd/single-socket-smd.kicad_pcb (KiCad board)
At the start: 2 copper layers, 97 x 96 mm, 278 parts, among them J109 Conn_01x01, J110 Conn_01x01, J111 Conn_01x01, J112 Conn_01x01, J113 Conn_01x01, J114 Conn_01x01, J115 Conn_01x01, J116 Conn_01x01, J117 Conn_01x01, J118 Conn_01x01, J119 Conn_01x01, J120 Conn_01x01, J121 Conn_01x01, J122 Conn_01x01, J123 Conn_01x01, J124 Conn_01x01, J125 Conn_01x01, J126 Conn_01x01, J127 Conn_01x01, J128 Conn_01x01, J129 Conn_01x01, J13 Conn_01x01, J130 Conn_01x01, J131 Conn_01x01, J132 Conn_01x01, J133 Conn_01x01, J134 Conn_01x01, J135 Conn_01x01, J136 Conn_01x01, J137 Conn_01x01, J138 Conn_01x01, J139 Conn_01x01, J14 Conn_01x01, J140 Conn_01x01, J141 Conn_01x01, J142 Conn_01x01, J143 Conn_01x01, J144 Conn_01x01, J145 Conn_01x01, J146 Conn_01x01, J147 Conn_01x01, J148 Conn_01x01, J149 Conn_01x01, J15 Conn_01x01, J150 Conn_01x01, J151 Conn_01x01, J152 Conn_01x01, J153 Conn_01x01, J154 Conn_01x01, J155 Conn_01x01, J156 Conn_01x01, J157 Conn_01x01, J158 Conn_01x01, J159 Conn_01x01, J16 Conn_01x01, J160 Conn_01x01, J161 Conn_01x01, J162 Conn_01x01, J163 Conn_01x01, J164 Conn_01x01, J165 Conn_01x01, J166 Conn_01x01, J167 Conn_01x01, J168 Conn_01x01, J169 Conn_01x01, J17 Conn_01x01, J170 Conn_01x01, J171 Conn_01x01, J172 Conn_01x01, J173 Conn_01x01, J174 Conn_01x01, J175 Conn_01x01, J176 Conn_01x01, J177 Conn_01x01, J178 Conn_01x01, J179 Conn_01x01, J18 Conn_01x01, J180 Conn_01x01, J19 Conn_01x01, J20 Conn_01x01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

Commit message: ok.
Parts:
- moved J123 4.03 mm to (33.5, 58.5)
- moved J125 4.03 mm to (33.5, 75.0)
- moved J127 4.03 mm to (33.5, 91.5)
- moved J129 4.03 mm to (33.5, 108.0)
- moved J133 4.03 mm to (53.5, 58.5)
- moved J135 4.03 mm to (53.5, 75.0)
- moved J137 4.03 mm to (53.5, 91.5)
- moved J143 4.03 mm to (73.5, 58.5)
- moved J145 4.03 mm to (73.5, 75.0)
- moved J147 4.03 mm to (73.5, 91.5)
- moved J149 4.03 mm to (73.5, 108.0)
- moved J151 4.03 mm to (93.5, 42.0)
- moved J153 4.03 mm to (93.5, 58.5)
- moved J155 4.03 mm to (93.5, 75.0)
- moved J157 4.03 mm to (93.5, 91.5)
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Routing:
- net Net-(J85-Pad1): track 0.00 -> 204.4 mm
- net Net-(J109-Pad1): track 0.00 -> 204.4 mm
- net Net-(J13-Pad1): track 36.0 -> 207.5 mm
- net Net-(J37-Pad1): track 35.5 -> 204.4 mm
- net Net-(J61-Pad1): track 35.5 -> 204.4 mm
- net Net-(J171-Pad1): track 0.00 -> 101.3 mm
- net Net-(J125-Pad1): track 0.00 -> 101.3 mm
- net Net-(J127-Pad1): track 0.00 -> 101.3 mm
- net Net-(J129-Pad1): track 0.00 -> 101.3 mm
- net Net-(J123-Pad1): track 0.00 -> 101.3 mm
- net Net-(J121-Pad1): track 64.9 -> 101.3 mm
- net Net-(diode2-Pad2): track 0.00 -> 9.39 mm
- net Net-(diode6-Pad2): track 0.00 -> 9.39 mm
- net Net-(diode5-Pad2): track 0.00 -> 9.39 mm
- net Net-(diode4-Pad2): track 0.00 -> 9.39 mm
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
Commit message: i forgot what i did.
Parts:
- removed J119, J120, J171, J172, J173, J174, J175, J176, J177, J178, J179, J180, J23, J24, J47, J48, J71, J72, J95, J96: Conn_01x01, footprints:wirepad
- removed the Ref** at (51.5, 124.5)
- removed the Ref** at (48.5, 124.5)
- removed the Ref** at (68.5, 124.5)
- removed the Ref** at (71.5, 124.5)
- removed the Ref** at (88.5, 124.5)
- removed the Ref** at (91.5, 124.5)
- removed the Ref** at (111.5, 124.5)
- removed the Ref** at (108.5, 124.5)
- removed the Ref** at (125.5, 111.0)
- removed the Ref** at (45.5, 111.0)
- removed the Ref** at (105.5, 114.0)
- removed the Ref** at (45.5, 114.0)
- removed the Ref** at (105.5, 111.0)
- removed the Ref** at (125.5, 114.0)
- removed the Ref** at (65.5, 114.0)
- removed the Ref** at (65.5, 111.0)
- removed the Ref** at (85.5, 114.0)
- removed the Ref** at (85.5, 111.0)
- removed diode12, diode18, diode24, diode30, diode6: diode, footprints:diodesmd
- removed switch12, switch18, switch24, switch30, switch6: switch, footprints:1u-socket-minimal-flipped
- added J1: Conn_01x01, footprints:wirepad, F.Cu at (33.0, 45.0)
- added J10: Conn_01x01, footprints:wirepad, F.Cu at (113.0, 63.0)
- added J11: Conn_01x01, footprints:wirepad, F.Cu at (33.0, 81.0)
- added J12: Conn_01x01, footprints:wirepad, F.Cu at (53.0, 81.0)
- added J2: Conn_01x01, footprints:wirepad, F.Cu at (53.0, 45.0)
- added J25: Conn_01x01, footprints:wirepad, F.Cu at (73.0, 81.0)
- added J26: Conn_01x01, footprints:wirepad, F.Cu at (93.0, 81.0)
- added J27: Conn_01x01, footprints:wirepad, F.Cu at (113.0, 81.0)
- added J28: Conn_01x01, footprints:wirepad, F.Cu at (33.0, 99.0)
- added J29: Conn_01x01, footprints:wirepad, F.Cu at (53.0, 99.0)
- added J3: Conn_01x01, footprints:wirepad, F.Cu at (73.0, 45.0)
- added J30: Conn_01x01, footprints:wirepad, F.Cu at (73.0, 99.0)
- added J31: Conn_01x01, footprints:wirepad, F.Cu at (93.0, 99.0)
- added J32: Conn_01x01, footprints:wirepad, F.Cu at (113.0, 99.0)
- added J33: Conn_01x01, footprints:wirepad, F.Cu at (33.0, 117.0)
- added J34: Conn_01x01, footprints:wirepad, F.Cu at (53.0, 117.0)
- added J35: Conn_01x01, footprints:wirepad, F.Cu at (73.0, 117.0)
- added J36: Conn_01x01, footprints:wirepad, F.Cu at (93.0, 117.0)
- added J4: Conn_01x01, footprints:wirepad, F.Cu at (93.0, 45.0)
- added J49: Conn_01x01, footprints:wirepad, F.Cu at (113.0, 117.0)
- added J5: Conn_01x01, footprints:wirepad, F.Cu at (113.0, 45.0)
- added J6: Conn_01x01, footprints:wirepad, F.Cu at (33.0, 63.0)
- added J7: Conn_01x01, footprints:wirepad, F.Cu at (53.0, 63.0)
- added J8: Conn_01x01, footprints:wirepad, F.Cu at (73.0, 63.0)
- added J9: Conn_01x01, footprints:wirepad, F.Cu at (93.0, 63.0)
- moved J118 8.08 mm to (127.0, 117.0)
- moved J22 8.08 mm to (47.0, 117.0)
- moved J46 8.08 mm to (67.0, 117.0)
- moved J70 8.08 mm to (87.0, 117.0)
- moved J94 8.08 mm to (107.0, 117.0)
- moved diode11 7.65 mm to (60.0, 116.5)
- moved diode17 7.65 mm to (80.0, 116.5)
- moved diode23 7.65 mm to (100.0, 116.5)
- moved diode29 7.65 mm to (120.0, 116.5)
- moved diode5 7.65 mm to (40.0, 116.5)
- moved J116 6.71 mm to (127.0, 99.0)
- moved J20 6.71 mm to (47.0, 99.0)
- moved J44 6.71 mm to (67.0, 99.0)
- moved J68 6.71 mm to (87.0, 99.0)
- moved J92 6.71 mm to (107.0, 99.0)
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Connections:
- J109 pad 1: Net-(J109-Pad1) -> Net-(J10-Pad1)
- J110 pad 1: Net-(J109-Pad1) -> Net-(J10-Pad1)
- J111 pad 1: Net-(J109-Pad1) -> Net-(J10-Pad1)
- J112 pad 1: Net-(J109-Pad1) -> Net-(J10-Pad1)
- J113 pad 1: Net-(J109-Pad1) -> Net-(J10-Pad1)
- J114 pad 1: Net-(J109-Pad1) -> Net-(J10-Pad1)
- J115 pad 1: Net-(J109-Pad1) -> Net-(J10-Pad1)
- J116 pad 1: Net-(J109-Pad1) -> Net-(J10-Pad1)
- J117 pad 1: Net-(J109-Pad1) -> Net-(J10-Pad1)
- J118 pad 1: Net-(J109-Pad1) -> Net-(J10-Pad1)
- J13 pad 1: Net-(J13-Pad1) -> Net-(J1-Pad1)
- J14 pad 1: Net-(J13-Pad1) -> Net-(J1-Pad1)
- J15 pad 1: Net-(J13-Pad1) -> Net-(J1-Pad1)
- J16 pad 1: Net-(J13-Pad1) -> Net-(J1-Pad1)
- J17 pad 1: Net-(J13-Pad1) -> Net-(J1-Pad1)
- J18 pad 1: Net-(J13-Pad1) -> Net-(J1-Pad1)
- J19 pad 1: Net-(J13-Pad1) -> Net-(J1-Pad1)
- J20 pad 1: Net-(J13-Pad1) -> Net-(J1-Pad1)
- J21 pad 1: Net-(J13-Pad1) -> Net-(J1-Pad1)
- J22 pad 1: Net-(J13-Pad1) -> Net-(J1-Pad1)
- J37 pad 1: Net-(J37-Pad1) -> Net-(J12-Pad1)
- J38 pad 1: Net-(J37-Pad1) -> Net-(J12-Pad1)
- J39 pad 1: Net-(J37-Pad1) -> Net-(J12-Pad1)
- J40 pad 1: Net-(J37-Pad1) -> Net-(J12-Pad1)
- J41 pad 1: Net-(J37-Pad1) -> Net-(J12-Pad1)
- J42 pad 1: Net-(J37-Pad1) -> Net-(J12-Pad1)
- J43 pad 1: Net-(J37-Pad1) -> Net-(J12-Pad1)
- J44 pad 1: Net-(J37-Pad1) -> Net-(J12-Pad1)
- J45 pad 1: Net-(J37-Pad1) -> Net-(J12-Pad1)
- J46 pad 1: Net-(J37-Pad1) -> Net-(J12-Pad1)
- J61 pad 1: Net-(J61-Pad1) -> Net-(J25-Pad1)
- J62 pad 1: Net-(J61-Pad1) -> Net-(J25-Pad1)
- J63 pad 1: Net-(J61-Pad1) -> Net-(J25-Pad1)
- J64 pad 1: Net-(J61-Pad1) -> Net-(J25-Pad1)
- J65 pad 1: Net-(J61-Pad1) -> Net-(J25-Pad1)
- J66 pad 1: Net-(J61-Pad1) -> Net-(J25-Pad1)
- J67 pad 1: Net-(J61-Pad1) -> Net-(J25-Pad1)
- J68 pad 1: Net-(J61-Pad1) -> Net-(J25-Pad1)
- J69 pad 1: Net-(J61-Pad1) -> Net-(J25-Pad1)
- J70 pad 1: Net-(J61-Pad1) -> Net-(J25-Pad1)
- J85 pad 1: Net-(J85-Pad1) -> Net-(J26-Pad1)
- J86 pad 1: Net-(J85-Pad1) -> Net-(J26-Pad1)
- J87 pad 1: Net-(J85-Pad1) -> Net-(J26-Pad1)
- J88 pad 1: Net-(J85-Pad1) -> Net-(J26-Pad1)
- J89 pad 1: Net-(J85-Pad1) -> Net-(J26-Pad1)
- J90 pad 1: Net-(J85-Pad1) -> Net-(J26-Pad1)
- J91 pad 1: Net-(J85-Pad1) -> Net-(J26-Pad1)
- J92 pad 1: Net-(J85-Pad1) -> Net-(J26-Pad1)
- J93 pad 1: Net-(J85-Pad1) -> Net-(J26-Pad1)
- J94 pad 1: Net-(J85-Pad1) -> Net-(J26-Pad1)
- switch1 pad 1: Net-(diode1-Pad2) -> Net-(J1-Pad1)
- switch1 pad 2: Net-(J13-Pad1) -> Net-(diode1-Pad2)
- switch10 pad 1: Net-(diode10-Pad2) -> Net-(J12-Pad1)
- switch10 pad 2: Net-(J37-Pad1) -> Net-(diode10-Pad2)
- switch11 pad 1: Net-(diode11-Pad2) -> Net-(J12-Pad1)
- switch11 pad 2: Net-(J37-Pad1) -> Net-(diode11-Pad2)
- switch13 pad 1: Net-(diode13-Pad2) -> Net-(J25-Pad1)
- switch13 pad 2: Net-(J61-Pad1) -> Net-(diode13-Pad2)
- switch14 pad 1: Net-(diode14-Pad2) -> Net-(J25-Pad1)
- switch14 pad 2: Net-(J61-Pad1) -> Net-(diode14-Pad2)
- switch15 pad 1: Net-(diode15-Pad2) -> Net-(J25-Pad1)
- switch15 pad 2: Net-(J61-Pad1) -> Net-(diode15-Pad2)
- switch16 pad 1: Net-(diode16-Pad2) -> Net-(J25-Pad1)
- switch16 pad 2: Net-(J61-Pad1) -> Net-(diode16-Pad2)
- switch17 pad 1: Net-(diode17-Pad2) -> Net-(J25-Pad1)
- switch17 pad 2: Net-(J61-Pad1) -> Net-(diode17-Pad2)
- switch19 pad 1: Net-(diode19-Pad2) -> Net-(J26-Pad1)
- switch19 pad 2: Net-(J85-Pad1) -> Net-(diode19-Pad2)
- switch2 pad 1: Net-(diode2-Pad2) -> Net-(J1-Pad1)
- switch2 pad 2: Net-(J13-Pad1) -> Net-(diode2-Pad2)
- switch20 pad 1: Net-(diode20-Pad2) -> Net-(J26-Pad1)
- switch20 pad 2: Net-(J85-Pad1) -> Net-(diode20-Pad2)
- switch21 pad 1: Net-(diode21-Pad2) -> Net-(J26-Pad1)
- switch21 pad 2: Net-(J85-Pad1) -> Net-(diode21-Pad2)
- switch22 pad 1: Net-(diode22-Pad2) -> Net-(J26-Pad1)
- switch22 pad 2: Net-(J85-Pad1) -> Net-(diode22-Pad2)
- switch23 pad 1: Net-(diode23-Pad2) -> Net-(J26-Pad1)
- switch23 pad 2: Net-(J85-Pad1) -> Net-(diode23-Pad2)
- switch25 pad 1: Net-(diode25-Pad2) -> Net-(J10-Pad1)
- switch25 pad 2: Net-(J109-Pad1) -> Net-(diode25-Pad2)
- switch26 pad 1: Net-(diode26-Pad2) -> Net-(J10-Pad1)
- switch26 pad 2: Net-(J109-Pad1) -> Net-(diode26-Pad2)
- switch27 pad 1: Net-(diode27-Pad2) -> Net-(J10-Pad1)
- switch27 pad 2: Net-(J109-Pad1) -> Net-(diode27-Pad2)
- switch28 pad 1: Net-(diode28-Pad2) -> Net-(J10-Pad1)
- switch28 pad 2: Net-(J109-Pad1) -> Net-(diode28-Pad2)
- switch29 pad 1: Net-(diode29-Pad2) -> Net-(J10-Pad1)
- switch29 pad 2: Net-(J109-Pad1) -> Net-(diode29-Pad2)
- switch3 pad 1: Net-(diode3-Pad2) -> Net-(J1-Pad1)
- switch3 pad 2: Net-(J13-Pad1) -> Net-(diode3-Pad2)
- switch4 pad 1: Net-(diode4-Pad2) -> Net-(J1-Pad1)
- switch4 pad 2: Net-(J13-Pad1) -> Net-(diode4-Pad2)
- switch5 pad 1: Net-(diode5-Pad2) -> Net-(J1-Pad1)
- switch5 pad 2: Net-(J13-Pad1) -> Net-(diode5-Pad2)
- switch7 pad 1: Net-(diode7-Pad2) -> Net-(J12-Pad1)
- switch7 pad 2: Net-(J37-Pad1) -> Net-(diode7-Pad2)
- switch8 pad 1: Net-(diode8-Pad2) -> Net-(J12-Pad1)
- switch8 pad 2: Net-(J37-Pad1) -> Net-(diode8-Pad2)
- switch9 pad 1: Net-(diode9-Pad2) -> Net-(J12-Pad1)
- switch9 pad 2: Net-(J37-Pad1) -> Net-(diode9-Pad2)
Routing:
- net Net-(J12-Pad1): track 0.00 -> 436.3 mm
- net Net-(J1-Pad1): track 0.00 -> 436.3 mm
- net Net-(J26-Pad1): track 0.00 -> 436.3 mm
- net Net-(J25-Pad1): track 0.00 -> 436.3 mm
- net Net-(J10-Pad1): track 0.00 -> 436.3 mm
- net Net-(J13-Pad1): track 207.5 -> 0.00 mm
- net Net-(J37-Pad1): track 204.4 -> 0.00 mm
- net Net-(J85-Pad1): track 204.4 -> 0.00 mm
- net Net-(J61-Pad1): track 204.4 -> 0.00 mm
- net Net-(J109-Pad1): track 204.4 -> 0.00 mm
- net Net-(J129-Pad1): track 101.3 -> 230.6 mm
- net Net-(J125-Pad1): track 101.3 -> 230.6 mm
- net Net-(J123-Pad1): track 101.3 -> 230.6 mm
- net Net-(J127-Pad1): track 101.3 -> 230.1 mm
- net Net-(J121-Pad1): track 101.3 -> 229.8 mm
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- added copper zone on B.Cu, net (none)
- added copper zone on F.Cu, net (none)
Other:
- board size 97 x 96 mm -> 97 x 87 mm
