File: socketsmd/single-socket-smd.sch (KiCad schematic (older format))
At the start: 180 parts, among them J109 Conn_01x01, J110 Conn_01x01, J111 Conn_01x01, J112 Conn_01x01, J113 Conn_01x01, J114 Conn_01x01, J115 Conn_01x01, J116 Conn_01x01, J117 Conn_01x01, J118 Conn_01x01, J119 Conn_01x01, J120 Conn_01x01, J121 Conn_01x01, J122 Conn_01x01, J123 Conn_01x01, J124 Conn_01x01, J125 Conn_01x01, J126 Conn_01x01, J127 Conn_01x01, J128 Conn_01x01, J129 Conn_01x01, J13 Conn_01x01, J130 Conn_01x01, J131 Conn_01x01, J132 Conn_01x01, J133 Conn_01x01, J134 Conn_01x01, J135 Conn_01x01, J136 Conn_01x01, J137 Conn_01x01, J138 Conn_01x01, J139 Conn_01x01, J14 Conn_01x01, J140 Conn_01x01, J141 Conn_01x01, J142 Conn_01x01, J143 Conn_01x01, J144 Conn_01x01, J145 Conn_01x01, J146 Conn_01x01, J147 Conn_01x01, J148 Conn_01x01, J149 Conn_01x01, J15 Conn_01x01, J150 Conn_01x01, J151 Conn_01x01, J152 Conn_01x01, J153 Conn_01x01, J154 Conn_01x01, J155 Conn_01x01, J156 Conn_01x01, J157 Conn_01x01, J158 Conn_01x01, J159 Conn_01x01, J16 Conn_01x01, J160 Conn_01x01, J161 Conn_01x01, J162 Conn_01x01, J163 Conn_01x01, J164 Conn_01x01, J165 Conn_01x01, J166 Conn_01x01, J167 Conn_01x01, J168 Conn_01x01, J169 Conn_01x01, J17 Conn_01x01, J170 Conn_01x01, J171 Conn_01x01, J172 Conn_01x01, J173 Conn_01x01, J174 Conn_01x01, J175 Conn_01x01, J176 Conn_01x01, J177 Conn_01x01, J178 Conn_01x01, J179 Conn_01x01, J18 Conn_01x01, J180 Conn_01x01, J19 Conn_01x01, J20 Conn_01x01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

Commit message: i forgot what i did.
Parts:
- removed J119, J120, J171, J172, J173, J174, J175, J176, J177, J178, J179, J180, J23, J24, J47, J48, J71, J72, J95, J96: Conn_01x01, footprints:wirepad, symbol Connector_Generic:Conn_01x01
- removed diode12, diode18, diode24, diode30, diode6: diode, footprints:diodesmd, symbol single:diode
- removed switch12, switch18, switch24, switch30, switch6: switch, footprints:1u-socket-minimal-flipped, symbol single:switch
- added J1, J10, J11, J12, J2, J25, J26, J27, J28, J29, J3, J30, J31, J32, J33, J34, J35, J36, J4, J49, J5, J6, J7, J8, J9: Conn_01x01, footprints:wirepad, symbol Connector_Generic:Conn_01x01
Connections:
- net at switch1.1: now also J13.1 (Pin_1), J14.1 (Pin_1), J15.1 (Pin_1), J16.1 (Pin_1), J17.1 (Pin_1), J18.1 (Pin_1), J19.1 (Pin_1), J20.1 (Pin_1), J21.1 (Pin_1), J22.1 (Pin_1), switch2.1, switch3.1, switch4.1, switch5.1, J1.1 (Pin_1), J11.1 (Pin_1), J28.1 (Pin_1), J33.1 (Pin_1), J6.1 (Pin_1); no longer diode1.2
- net at diode2.2: now also switch2.2; no longer switch2.1
- net at diode3.2: now also switch3.2; no longer switch3.1
- net at diode4.2: now also switch4.2; no longer switch4.1
- net at diode5.2: now also switch5.2; no longer switch5.1
- net at diode7.2: now also switch7.2; no longer switch7.1
- net at J37.1 (Pin_1), J38.1 (Pin_1), J39.1 (Pin_1)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: now also switch10.1, switch11.1, switch7.1, switch8.1, switch9.1, J12.1 (Pin_1), J2.1 (Pin_1), J29.1 (Pin_1), J34.1 (Pin_1), J7.1 (Pin_1); no longer switch10.2, switch11.2, switch7.2, switch8.2, switch9.2
- net at diode8.2: now also switch8.2; no longer switch8.1
- net at diode9.2: now also switch9.2; no longer switch9.1
- net at diode10.2: now also switch10.2; no longer switch10.1
- net at diode11.2: now also switch11.2; no longer switch11.1
- net at diode13.2: now also switch13.2; no longer switch13.1
- net at J61.1 (Pin_1), J62.1 (Pin_1), J63.1 (Pin_1)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: now also switch13.1, switch14.1, switch15.1, switch16.1, switch17.1, J25.1 (Pin_1), J3.1 (Pin_1), J30.1 (Pin_1), J35.1 (Pin_1), J8.1 (Pin_1); no longer switch13.2, switch14.2, switch15.2, switch16.2, switch17.2
- net at diode14.2: now also switch14.2; no longer switch14.1
- net at diode15.2: now also switch15.2; no longer switch15.1
- net at diode16.2: now also switch16.2; no longer switch16.1
- net at diode17.2: now also switch17.2; no longer switch17.1
- net at diode19.2: now also switch19.2; no longer switch19.1
- net at J85.1 (Pin_1), J86.1 (Pin_1), J87.1 (Pin_1)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: now also switch19.1, switch20.1, switch21.1, switch22.1, switch23.1, J26.1 (Pin_1), J31.1 (Pin_1), J36.1 (Pin_1), J4.1 (Pin_1), J9.1 (Pin_1); no longer switch19.2, switch20.2, switch21.2, switch22.2, switch23.2
- net at diode20.2: now also switch20.2; no longer switch20.1
- net at diode21.2: now also switch21.2; no longer switch21.1
- net at diode22.2: now also switch22.2; no longer switch22.1
- net at diode23.2: now also switch23.2; no longer switch23.1
- net at diode25.2: now also switch25.2; no longer switch25.1
- net at J109.1 (Pin_1), J110.1 (Pin_1), J111.1 (Pin_1)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: now also switch25.1, switch26.1, switch27.1, switch28.1, switch29.1, J10.1 (Pin_1), J27.1 (Pin_1), J32.1 (Pin_1), J49.1 (Pin_1), J5.1 (Pin_1); no longer switch25.2, switch26.2, switch27.2, switch28.2, switch29.2
- net at diode26.2: now also switch26.2; no longer switch26.1
- net at diode27.2: now also switch27.2; no longer switch27.1
- net at diode28.2: now also switch28.2; no longer switch28.1
- net at diode29.2: now also switch29.2; no longer switch29.1
- new net: diode1.2, switch1.2
Other:
- moved on the sheet: switch1, switch10, switch11, switch13, switch14, switch15, switch16, switch17, switch19, switch2, switch20, switch21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
