File: choc-socket/single-choc-socket.kicad_pcb (KiCad board)
At the start: 2 copper layers, 97 x 117 mm, 339 parts, among them J1 Conn_01x01, J10 Conn_01x01, J100 Conn_01x01, J101 Conn_01x01, J102 Conn_01x01, J103 Conn_01x01, J104 Conn_01x01, J105 Conn_01x01, J106 Conn_01x01, J107 Conn_01x01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

Commit message: zone.
Routing:
- added copper zone on B.Cu, net (none)
- added copper zone on F.Cu, net (none)
